Commit message: chore(description): gazebo sim plugin updated

File: waver_description/urdf/depth_camera_zedxm.xacro (robot description, xacro)
@@ -36,7 +36,8 @@
     <gazebo reference="zed_x_mini_link">
         <material>Gazebo/Black</material>
-        <sensor name="depth" type="depth">
+        <sensor name="depth" type="depth_camera">
             <visualize>true</visualize>
             <update_rate>60.0</update_rate>
+            <topic>depth_camera</topic>
             <camera>
                 <horizontal_fov>1.047198</horizontal_fov>
@@ -56,22 +57,4 @@
                 </noise>
             </camera>
-            <plugin name="depth_camera_controller" filename="libgazebo_ros_camera.so">
-                <baseline>0.05</baseline>
-                <alwaysOn>true</alwaysOn>
-                <updateRate>60.0</updateRate>
-                <frame_name>zed_x_mini_optical_frame</frame_name>
-                <pointCloudCutoff>0.1</pointCloudCutoff>
-                <pointCloudCutoffMax>8.0</pointCloudCutoffMax>
-                <distortionK1>0</distortionK1>
-                <distortionK2>0</distortionK2>
-                <distortionK3>0</distortionK3>
-                <distortionT1>0</distortionT1>
-                <distortionT2>0</distortionT2>
-                <CxPrime>0</CxPrime>
-                <Cx>0</Cx>
-                <Cy>0</Cy>
-                <focalLength>0</focalLength>
-                <hackBaseline>0</hackBaseline>
-            </plugin>
         </sensor>
     </gazebo>

File: waver_description/urdf/imu.xacro (robot description, xacro)
@@ -36,15 +36,4 @@
             <visualize>true</visualize>
             <topic>imu</topic>
-            <plugin filename="libgazebo_ros_imu_sensor.so" name="imu">
-                <topicName>imu</topicName>
-                <bodyName>imu_link</bodyName>
-                <updateRateHZ>10.0</updateRateHZ>
-                <gaussianNoise>0.0</gaussianNoise>
-                <xyzOffset>0 0 0</xyzOffset>
-                <rpyOffset>0 0 0</rpyOffset>
-                <frameName>imu_link</frameName>
-                <initialOrientationAsReference>false</initialOrientationAsReference>
-            </plugin>
-            <pose>0 0 0 0 0 0</pose>
         </sensor>
     </gazebo>

File: waver_description/urdf/lidar.xacro (robot description, xacro)
@@ -30,5 +30,5 @@
     <gazebo reference="${lidar_link}">
         <material>Gazebo/Black</material>
-        <sensor name="${lidar_model}" type="ray">
+        <sensor name="${lidar_model}" type="gpu_lidar">
             <pose>0 0 0 0 0 0</pose>
             <visualize>false</visualize>
@@ -40,4 +40,5 @@
                     <horizontal>
                         <samples>${lidar_samples}</samples>
+                        <resolution>1</resolution>
                         <min_angle>${lidar_min_angle}</min_angle>
                         <max_angle>${lidar_max_angle}</max_angle>
@@ -47,4 +48,5 @@
                     <min>${lidar_min_range}</min>
                     <max>${lidar_max_range}</max>
+                    <resolution>0.01</resolution>
                 </range>
                 <noise>
@@ -54,12 +56,4 @@
                 </noise>
             </ray>
-            <plugin name="lidar_controller" filename="libgazebo_ros_ray_sensor.so">
-                <ros>
-                    <namespace>/</namespace>
-                    <remapping>~/out:=scan</remapping>
-                </ros>
-                <output_type>sensor_msgs/LaserScan</output_type>
-                <frame_name>${lidar_link}</frame_name>
-            </plugin>
         </sensor>
     </gazebo>

File: waver_description/urdf/rasp_pi_camera.xacro (robot description, xacro)
@@ -7,10 +7,12 @@
             <mass value="${rasp_pi_camera_mass}" />
             <origin xyz="0 0 0" rpy="0 0 0" />
-            <inertia ixx="8.188544198245058e-07" iyy="1.3934609636775025e-06" izz="8.837267894803364e-07" ixy="0" iyz="0" ixz="0" />
+            <inertia ixx="8.188544198245058e-07" iyy="1.3934609636775025e-06"
+                izz="8.837267894803364e-07" ixy="0" iyz="0" ixz="0" />
         </inertial>
         <visual>
             <origin xyz="0 0.0125 0" rpy="0 0 ${-pi/2}" />
             <geometry>
-                <mesh filename="file:///$(find waver_description)/meshes/rasp_pi_camera.stl" scale="${camera_scale}" />
+                <mesh filename="package://waver_description/meshes/rasp_pi_camera.stl"
+                    scale="${camera_scale}" />
             </geometry>
             <xacro:black_material />
@@ -19,5 +21,6 @@
             <origin xyz="0 0.0125 0" rpy="0 0 ${-pi/2}" />
             <geometry>
-                <mesh filename="file:///$(find waver_description)/meshes/rasp_pi_camera.stl" scale="${camera_scale}" />
+                <mesh filename="package://waver_description/meshes/rasp_pi_camera.stl"
+                    scale="${camera_scale}" />
             </geometry>
         </collision>
@@ -34,10 +37,11 @@
             <visualize>false</visualize>
             <update_rate>30</update_rate>
+            <topic>image_raw</topic>
             <camera>
                 <horizontal_fov>1.1519</horizontal_fov>
                 <image>
                     <format>R8G8B8</format>
-                    <width>4608</width>
-                    <height>2592</height>
+                    <height>1080</height>
+                    <width>1920</width>
                 </image>
                 <clip>
@@ -51,18 +55,4 @@
                 </noise>
             </camera>
-            <plugin name="camera_controller" filename="libgazebo_ros_camera.so">
-                <alwaysOn>true</alwaysOn>
-                <updateRate>30</updateRate>
-                <cameraName>camera</cameraName>
-                <imageTopicName>image_raw</imageTopicName>
-                <cameraInfoTopicName>camera_info</cameraInfoTopicName>
-                <frameName>rasp_pi_camera_link</frameName>
-                <hackBaseline>0.07</hackBaseline>
-                <distortionK1>0.0</distortionK1>
-                <distortionK2>0.0</distortionK2>
-                <distortionK3>0.0</distortionK3>
-                <distortionT1>0.0</distortionT1>
-                <distortionT2>0.0</distortionT2>
-            </plugin>
         </sensor>
     </gazebo>

File: waver_description/urdf/waver.gazebo.xacro (robot description, xacro)
@@ -63,6 +63,5 @@
   </gazebo>
   <gazebo>
-    <plugin
-      filename="gz-sim-diff-drive-system" name="gz::sim::systems::DiffDrive">
+    <plugin filename="libgz-sim-diff-drive-system.so" name="gz::sim::systems::DiffDrive">
       <left_joint>wheel_front_left_joint</left_joint>
       <right_joint>wheel_front_right_joint</right_joint>
@@ -82,7 +81,10 @@
       <odom_publish_frequency>30</odom_publish_frequency>
     </plugin>
-    <plugin
-      filename="gz-sim-joint-state-publisher-system" name="gz::sim::systems::JointStatePublisher">
+    <plugin filename="libgz-sim-joint-state-publisher-system.so"
+      name="gz::sim::systems::JointStatePublisher">
       <topic>joint_states</topic>
+    </plugin>
+    <plugin filename="libgz-sim-sensors-system.so" name="gz::sim::systems::Sensors">
+      <render_engine>ogre2</render_engine>
     </plugin>
   </gazebo>

Commit message: chore(descr): ros2_control implementation added

File: waver_description/urdf/depth_camera_zedxm.xacro (robot description, xacro)
@@ -12,5 +12,5 @@
             <origin xyz="0 0 0" rpy="0 0 0" />
             <geometry>
-                <mesh filename="file:///$(find waver_description)/meshes/zedxm.stl" scale="${zed_x_mini_scale}" />
+                <mesh filename="package://waver_description/meshes/zedxm.stl" scale="${zed_x_mini_scale}" />
             </geometry>
             <xacro:black_material />
@@ -19,5 +19,5 @@
             <origin xyz="0 0 0" rpy="0 0 0" />
             <geometry>
-                <mesh filename="file:///$(find waver_description)/meshes/zedxm.stl" scale="${zed_x_mini_scale}" />
+                <mesh filename="package://waver_description/meshes/zedxm.stl" scale="${zed_x_mini_scale}" />
             </geometry>
         </collision>

File: waver_description/urdf/waver.xacro (robot description, xacro)
@@ -1,11 +1,18 @@
 <?xml version="1.0"?>
 <robot name="waver" xmlns:xacro="http://www.ros.org/wiki/xacro">
+  <xacro:arg name="sim_control" default="gazebo" />
   <xacro:arg name="camera_type" default="raspi" />
   <xacro:include filename="$(find waver_description)/urdf/materials.xacro" />
   <xacro:include filename="$(find waver_description)/urdf/util.xacro" />
-  <xacro:include filename="$(find waver_description)/urdf/waver.trans.xacro" />
-  <xacro:include filename="$(find waver_description)/urdf/waver.gazebo.xacro" />
   <xacro:include filename="$(find waver_description)/urdf/lidar.xacro" />
   <xacro:include filename="$(find waver_description)/urdf/imu.xacro" />
+  <!-- ************************** Simulation Control ************************** -->
+  <xacro:if value="${'$(arg sim_control)' == 'gazebo'}">
+    <xacro:include filename="$(find waver_description)/urdf/waver.gazebo.xacro" />
+  </xacro:if>
+  <xacro:if value="${'$(arg sim_control)' == 'ros2'}">
+    <xacro:include filename="$(find waver_description)/urdf/waver.control.xacro" />
+  </xacro:if>
+  <!-- ***************************** Camera Type ***************************** -->
   <xacro:if value="${'$(arg camera_type)' == 'raspi'}">
     <xacro:include filename="$(find waver_description)/urdf/rasp_pi_camera.xacro" />
