Commit message: fix(descr): wheel collitions updated to improve performance

File: waver_description/urdf/util.xacro (robot description, xacro)
@@ -57,4 +57,5 @@
     <xacro:property name="wheel_separation" value="123e-3" />
     <xacro:property name="wheel_radius" value="40.6e-3" />
+    <xacro:property name="wheel_width" value="42.5e-3" />
     <!-- WBL specifications -->
     <xacro:property name="pos_x_wbl" value="0.06538582611083985" />

File: waver_description/urdf/waver.xacro (robot description, xacro)
@@ -144,8 +144,7 @@
     </visual>
     <collision>
-      <origin xyz="${position_wbl}" rpy="0 0 ${pi/2}" />
-      <geometry>
-        <mesh filename="package://waver_description/meshes/wheel_back_left_link.stl"
-          scale="${scale}" />
+      <origin xyz="0 0 0" rpy="${pi/2} 0 0" />
+      <geometry>
+        <cylinder radius="${wheel_radius}" length="${wheel_width}" />
       </geometry>
     </collision>
@@ -167,8 +166,7 @@
     </visual>
     <collision>
-      <origin xyz="${position_wfl}" rpy="0 0 ${pi/2}" />
-      <geometry>
-        <mesh filename="package://waver_description/meshes/wheel_front_left_link.stl"
-          scale="${scale}" />
+      <origin xyz="0 0 0" rpy="${pi/2} 0 0" />
+      <geometry>
+        <cylinder radius="${wheel_radius}" length="${wheel_width}" />
       </geometry>
     </collision>
@@ -190,8 +188,7 @@
     </visual>
     <collision>
-      <origin xyz="${position_wfr}" rpy="0 0 ${pi/2}" />
-      <geometry>
-        <mesh filename="package://waver_description/meshes/wheel_front_right_link.stl"
-          scale="${scale}" />
+      <origin xyz="0 0 0" rpy="${pi/2} 0 0" />
+      <geometry>
+        <cylinder radius="${wheel_radius}" length="${wheel_width}" />
       </geometry>
     </collision>
@@ -213,8 +210,7 @@
     </visual>
     <collision>
-      <origin xyz="${position_wbr}" rpy="0 0 ${pi/2}" />
-      <geometry>
-        <mesh filename="package://waver_description/meshes/wheel_back_right_link.stl"
-          scale="${scale}" />
+      <origin xyz="0 0 0" rpy="${pi/2} 0 0" />
+      <geometry>
+        <cylinder radius="${wheel_radius}" length="${wheel_width}" />
       </geometry>
     </collision>
