Commit message: Refactor robot control files and add new nodes for improved functionality and integration with MoveIt. Update URDF configurations for Gazebo compatibility, implement ArUco marker detection, and enhance gripper control logic. Introduce launch files for streamlined execution of pick and place operations.

File: wave_rover/waver_description/urdf/waver.control.xacro (robot description, xacro)
@@ -75,5 +75,5 @@
     <ros2_control name="waver" type="system">
         <hardware>
-            <plugin>gz_ros2_control/GazeboSimSystem</plugin>
+            <plugin>gz_ros2_control/GazeboSystem</plugin>
         </hardware>
         <joint name="wheel_front_left_joint">

File: wave_rover/waver_description/urdf/waver.xacro (robot description, xacro)
@@ -261,4 +261,29 @@
     <axis xyz="0 1 0" />
   </joint>
+    <ros2_control name="waver" type="system">
+    <hardware>
+      <plugin>gz_ros2_control/GazeboSystem</plugin>
+    </hardware>
+    <joint name="wheel_front_left_joint">
+      <command_interface name="velocity"/>
+      <state_interface name="position"/>
+      <state_interface name="velocity"/>
+    </joint>
+    <joint name="wheel_front_right_joint">
+      <command_interface name="velocity"/>
+      <state_interface name="position"/>
+      <state_interface name="velocity"/>
+    </joint>
+    <joint name="wheel_back_left_joint">
+      <command_interface name="velocity"/>
+      <state_interface name="position"/>
+      <state_interface name="velocity"/>
+    </joint>
+    <joint name="wheel_back_right_joint">
+      <command_interface name="velocity"/>
+      <state_interface name="position"/>
+      <state_interface name="velocity"/>
+    </joint>
+  </ros2_control>
   <joint name="wheel_back_right_joint" type="continuous">
     <origin xyz="${position_wbr_joint}" rpy="0 0 0" />
